Commit message: feat: add nav configs and nav image build as well as simualtion fixes

File: simulated_turtlebot/rplidar.urdf.xacro (robot description, xacro)
@@ -29,5 +29,35 @@
     <xacro:inertial_cuboid mass="0.17" x="${length_x}" y="${length_y}" z="${length_z}"/>
   </link>
-  <gazebo reference="${name}_link">
+    <gazebo reference="${name}_link">
+      <!--<material>
+        <ambient>${gazebo_material_ambient}</ambient>
+        <diffuse>${gazebo_material_diffuse}</diffuse>
+        <specular>${gazebo_material_specular}</specular>
+      </material> -->
+      <!-- GPU ray sensors run in the rendering, so they are usually more efficient and detect visual shapes. -->
+      <!-- Ray sensors run in the physics, so they're less efficient and detect collision shapes. -->
+      <sensor name='${name}' type='gpu_lidar'>
+        <update_rate>12</update_rate>
+        <always_on>1</always_on>
+        <visualize>1</visualize>
+        <ray>
+          <scan>
+            <horizontal>
+              <samples>640</samples>
+              <resolution>1</resolution>
+              <min_angle>${-pi}</min_angle>
+              <max_angle>${pi}</max_angle>
+            </horizontal>
+          </scan>
+          <range>
+            <min>0.164</min>
+            <max>12.0</max>
+            <resolution>0.01</resolution>
+          </range>
+        </ray>
+        <gz_frame_id>${name}_link</gz_frame_id>
+      </sensor>
+    </gazebo>
+  <!-- <gazebo reference="${name}_link">
     <xacro:ray_sensor sensor_name="${name}" gazebo="${gazebo}"
                   update_rate="20.0" visualize="0"
@@ -37,5 +67,5 @@
     </xacro:ray_sensor>
     <xacro:material_darkgray/>
-  </gazebo>
+  </gazebo> -->
   <gazebo reference="${name}_joint">
     <preserveFixedJoint>true</preserveFixedJoint>
